File: 433/mini_tracker.kicad_sch (KiCad schematic)
At the start: 32 parts, among them J2 Conn_01x05_Male, SW1 SW_DIP_x03, U2 AP2210N-3.3TRG1, U3 STM32G030F6P6, U4 SIM28ML, Y2 NX2016SA-32MHZ-STD-CZS-5

Commit message: Update production files
-Fixed sta and pps label swap for both versions
-Completely redesign passive network for 868 version for lower extended components fee
Parts:
- AE1, BT1, J2, JP1, TP1: now left out of the parts list
