File: 433/sx1262.kicad_sch (KiCad schematic)
At the start: 31 parts, among them J1 Conn_Coaxial, U1 SX1262, U5 SKY13453-385LF, Y1 NX2016SA-32MHZ-STD-CZS-5

Commit message: Update production files
-Fixed sta and pps label swap for both versions
-Completely redesign passive network for 868 version for lower extended components fee
Parts:
- C23, C24: now not fitted
- J1: now left out of the parts list
