File: 868_915/sx1262.kicad_sch (KiCad schematic)
At the start: 31 parts, among them J1 Conn_Coaxial, U1 SX1262, U5 SKY13453-385LF, Y1 NX2016SA-32MHZ-STD-CZS-5

Commit message: Update production files
-Fixed sta and pps label swap for both versions
-Completely redesign passive network for 868 version for lower extended components fee
Parts:
- removed C12: 1pF, Capacitor_SMD:C_0402_1005Metric, symbol Device:C
- removed C13: 47pF, Capacitor_SMD:C_0402_1005Metric, symbol Device:C
- added L7: 1.3nH, Inductor_SMD:L_0402_1005Metric, symbol Device:L
- added L8: 12nH, Inductor_SMD:L_0402_1005Metric, symbol Device:L
- C11: value 3.6pF -> 1.5pF; LCSC C52052 -> C1552
- C19: value 15pF -> 5.6pF; LCSC C1548 -> C1574
- C21: value 9pF -> 5.6pF; LCSC C126519 -> C1574
- C22: value 22pF -> 100pF; LCSC C1562 -> C1546
- C23, C24: now not fitted
- C9: value 2.7pF -> 5.6pF; LCSC C172851 -> C1574
- J1: now left out of the parts list
- L4: value 9.1nH -> 6.5nH; LCSC C142211 -> C778787
- L5: value 4.3nH -> 12nH; LCSC C395069 -> C275264
Connections:
- net GND: no longer C21.1
- net at C9.2, U1.21 (RFI_P): now also L8.2; no longer L3.2
- net at C20.1: now also C21.1, L7.2; no longer L5.2
- net at C20.2, U5.2 (RF1): no longer C21.2
- new net: L3.2, L8.1
- new net: C21.2, L5.2, L7.1
Other:
- moved on the sheet: C19, C20, C21, C9, L4, L5
